File: switch/_autosave-switch.kicad_sch (KiCad schematic)
At the start: 0 parts

Commit message: Working on PSU's
Other:
- added sheet SW_PSU (SW_PSU.kicad_sch)
Changed lines of the file:
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@@
+    (stroke (width 0) (type default))
+  )
+  (wire (pts (xy 179.07 77.47) (xy 179.07 83.82))
     (stroke (width 0) (type default))
   )
@@
     (effects (font (size 1.27 1.27)) (justify left bottom))
   )
+  (label "3.3V_PCIE" (at 353.06 96.52 90) (fields_autoplaced)
+    (effects (font (size 1.27 1.27)) (justify left bottom))
+  )
+  (label "3.3V_PCIE" (at 389.89 125.73 90) (fields_autoplaced)
+    (effects (font (size 1.27 1.27)) (justify left bottom))
+  )
+  (label "3.3V_PCIE" (at 179.07 77.47 90) (fields_autoplaced)
+    (effects (font (size 1.27 1.27)) (justify left bottom))
+  )
   (label "+12V_PCIE" (at 176.53 78.74 90) (fields_autoplaced)
     (effects (font (size 1.27 1.27)) (justify left bottom))
   )
+  (label "3.3V_PCIE" (at 218.44 52.07 90) (fields_autoplaced)
+    (effects (font (size 1.27 1.27)) (justify left bottom))
+  )
   (label "+12V_PCIE" (at 316.23 67.31 90) (fields_autoplaced)
+    (effects (font (size 1.27 1.27)) (justify left bottom))
+  )
+  (label "3.3V_PCIE" (at 320.04 67.31 90) (fields_autoplaced)
+    (effects (font (size 1.27 1.27)) (justify left bottom))
+  )
+  (label "3.3V_PCIE" (at 386.08 125.73 90) (fields_autoplaced)
+    (effects (font (size 1.27 1.27)) (justify left bottom))
+  )
+  (label "3.3V_PCIE" (at 323.85 67.31 90) (fields_autoplaced)
+    (effects (font (size 1.27 1.27)) (justify left bottom))
+  )
+  (label "3.3V_PCIE" (at 356.87 96.52 90) (fields_autoplaced)
     (effects (font (size 1.27 1.27)) (justify left bottom))
   )
@@
       )
     )
+  )
+  (sheet (at 250.19 20.32) (size 25.4 29.21) (fields_autoplaced)
+    (stroke (width 0.1524) (type solid))
+    (fill (color 0 0 0 0.0000))
+    (property "Sheetname" "SW_PSU" (at 250.19 19.6084 0)
+      (effects (font (size 1.27 1.27)) (justify left bottom))
+    )
+    (property "Sheetfile" "SW_PSU.kicad_sch" (at 250.19 50.1146 0)
+      (effects (font (size 1.27 1.27)) (justify left top))
+    )
+    (instances
+      (project "switch"
+        (path "/bb24befe-87e3-4bdd-b50d-d3887bf8bcae" (page "7"))
+      )
+    )
