File: switch/switch.kicad_pcb (KiCad board)
At the start: 2 copper layers, 8.4 x 20.3 mm, 81 parts, among them J1 Bus_PCI_Express_x1, U1 PI7C9X2G404SLBFDEX, U2 M24C04-WMN6TP

Commit message: Finished with Schematic.
Parts:
- added CN1: 3183-10110P1T, NEW:CONN-TH_36P-P1.00-V_3183-XXXXXPXT, F.Cu at (136.6, 62.6)
Connections:
- J1 pad A11: /PCIE_UPSTREAM/PCIE_N_RESET -> /PCIE_SWITCH/PERST_L
- J1 pad A13: /PCIE_UPSTREAM/PCIE_REFCLK_P -> /PCIE_SWITCH/REFCLK(0)_N
- J1 pad A14: /PCIE_UPSTREAM/PCIE_REFCLK_N -> /PCIE_SWITCH/REFCLK(0)_P
- J1 pad A16: /PCIE_UPSTREAM/PCIE_RX_P -> /PCIE_SWITCH/PER(0)_P
- J1 pad A17: /PCIE_UPSTREAM/PCIE_RX_N -> /PCIE_SWITCH/PER(0)_N
- J1 pad B12: unconnected-(J1-RSVD-PadB12) -> /PCIE_SWITCH/CLOCKREQ_(0)
- J1 pad B14: /PCIE_UPSTREAM/PCIE_TX_P -> /PCIE_SWITCH/PCIE_RX_P
- J1 pad B15: /PCIE_UPSTREAM/PCIE_TX_N -> /PCIE_SWITCH/PCIE_RX_N
- L3 pad 2: /PCIE_SWITCH/+1.0V -> /PCIE_SWITCH/1.0Vaux
- L5 pad 2: /PCIE_SWITCH/3.3V_PCIE -> /PCIE_SWITCH/3.3Vaux

Commit message: Working on layout.
Parts:
- added C49: 1u, Capacitor_SMD:C_0402_1005Metric, F.Cu at (169.4, 57.8)
- added C50: 1u, Capacitor_SMD:C_0402_1005Metric, F.Cu at (169.4, 59.8)
- added C51: 1u, Capacitor_SMD:C_0402_1005Metric, F.Cu at (169.4, 61.8)
- added C52: 1u, Capacitor_SMD:C_0402_1005Metric, F.Cu at (169.4, 63.7)
- added C53: 1u, Capacitor_SMD:C_0402_1005Metric, F.Cu at (169.4, 65.7)
- added C54: 2.2u, Capacitor_SMD:C_0402_1005Metric, F.Cu at (169.4, 67.7)
- added C55: 1u, Capacitor_SMD:C_0402_1005Metric, F.Cu at (169.4, 69.7)
- added C56: 2.2u, Capacitor_SMD:C_0402_1005Metric, F.Cu at (169.4, 71.6)
- added CN2: 3183-10110P1T, NEW:CONN-TH_36P-P1.00-V_3183-XXXXXPXT, F.Cu at (227.2, 121.2)
- added CN3: 3183-10110P1T, NEW:CONN-TH_36P-P1.00-V_3183-XXXXXPXT, F.Cu at (254.6, 117.5)
- added LDO1: TPS70933DBVR, NEW:SOT-23-5_L3.0-W1.7-P0.95-LS2.8-BR, F.Cu at (173.2, 59.0)
- added LDO2: TPS70933DBVR, NEW:SOT-23-5_L3.0-W1.7-P0.95-LS2.8-BR, F.Cu at (173.2, 63.6)
- added U3: TLV73310PDBVR, NEW:TSOT-23-5_L2.9-W1.6-P0.95-LS2.8-BR, F.Cu at (177.8, 59.1)
- added U4: TLV73310PDBVR, NEW:TSOT-23-5_L2.9-W1.6-P0.95-LS2.8-BR, F.Cu at (177.8, 63.6)
- moved C20 118.2 mm to (187.8, 115.0)
- moved C24 114.9 mm to (187.7, 113.6)
- moved C10 111.1 mm to (167.4, 129.0), turned to 90 degrees
- moved C3 111.1 mm to (171.8, 118.5)
- moved L1 109.7 mm to (155.5, 135.4), turned to 90 degrees
- moved C7 109.2 mm to (171.8, 122.1), turned to 180 degrees
- moved C4 108.1 mm to (171.8, 113.3), turned to 180 degrees
- moved C6 106.2 mm to (171.8, 112.3)
- moved C9 104.8 mm to (158.2, 129.0), turned to -90 degrees
- moved L2 104.2 mm to (147.6, 136.6)
- moved U1 104.0 mm to (161.6, 118.7)
- moved C22 101.7 mm to (164.2, 129.0), turned to 90 degrees
- moved C19 101.1 mm to (159.4, 129.0), turned to -90 degrees
- moved R2 100.9 mm to (161.3, 137.9)
- moved C21 99.8 mm to (160.6, 129.0), turned to -90 degrees
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Connections:
- C36 pad 2: /PCIE_SWITCH/PCIe_TX_P(1) -> /PCIE_DOWNSTREAM1/PCIE_TX_P
- C37 pad 2: /PCIE_SWITCH/PCIe_TX_P(2) -> /PCIE_DOWNSTREAM2/PCIE_TX_P
- C38 pad 2: /PCIE_SWITCH/REFCLCK_N(2) -> /PCIE_DOWNSTREAM2/REF_CLK_N
- C39 pad 2: /PCIE_SWITCH/PCIe_TX_P(3) -> /PCIE_DOWNSTREAM3/PCIE_TX_P
- C40 pad 2: /PCIE_SWITCH/REFCLCK_N(3) -> /PCIE_DOWNSTREAM3/REF_CLK_N
- C41 pad 2: /PCIE_SWITCH/REFCLCK_N(1) -> /PCIE_DOWNSTREAM1/REF_CLK_N
- C42 pad 2: /PCIE_SWITCH/REFCLCK_P(2) -> /PCIE_DOWNSTREAM2/REF_CLK_P
- C43 pad 2: /PCIE_SWITCH/REFCLCK_P(3) -> /PCIE_DOWNSTREAM3/REF_CLK_P
- C44 pad 2: /PCIE_SWITCH/PCIe_TX_N(1) -> /PCIE_DOWNSTREAM1/PCIE_TX_N
- C45 pad 2: /PCIE_SWITCH/REFCLCK_P(1) -> /PCIE_DOWNSTREAM1/REF_CLK_P
- C46 pad 2: /PCIE_SWITCH/PCIe_TX_N(2) -> /PCIE_DOWNSTREAM2/PCIE_TX_N
- C47 pad 2: /PCIE_SWITCH/PCIe_TX_N(3) -> /PCIE_DOWNSTREAM3/PCIE_TX_N
- CN1 pad A10: /PCIE_DOWNSTREAM/+3.3V -> /3.3V_PCIE
- CN1 pad A11: /PCIE_DOWNSTREAM/PCIE_N_RESET -> /PCIE_SWITCH/DWNRST_L(1)
- CN1 pad A13: /PCIE_DOWNSTREAM/REF_CLK_P -> /PCIE_DOWNSTREAM1/REF_CLK_P
- CN1 pad A14: /PCIE_DOWNSTREAM/REF_CLK_N -> /PCIE_DOWNSTREAM1/REF_CLK_N
- CN1 pad A16: /PCIE_DOWNSTREAM/PCIE_RX_P -> /PCIE_SWITCH/PER(1)_P
- CN1 pad A17: /PCIE_DOWNSTREAM/PCIE_RX_N -> /PCIE_SWITCH/PER(1)_N
- CN1 pad A2: /PCIE_DOWNSTREAM/+12V -> /+12V_PCIE
- CN1 pad A3: /PCIE_DOWNSTREAM/+12V -> /+12V_PCIE
- CN1 pad A5: /PCIE_DOWNSTREAM/+3.3V -> /3.3V_PCIE
- CN1 pad A6: /PCIE_DOWNSTREAM/+3.3V -> /3.3V_PCIE
- CN1 pad A8: /PCIE_DOWNSTREAM/+3.3V -> /3.3V_PCIE
- CN1 pad A9: /PCIE_DOWNSTREAM/+3.3V -> /3.3V_PCIE
- CN1 pad B1: /PCIE_DOWNSTREAM/+12V -> /+12V_PCIE
- CN1 pad B10: /PCIE_DOWNSTREAM/+3.3VAux -> /3.3V_PCIE
- CN1 pad B12: /PCIE_DOWNSTREAM/PCIE_n_CLK_REQ -> /PCIE_SWITCH/CLOCKREQ_(1)
- CN1 pad B14: /PCIE_DOWNSTREAM/PCIE_TX_P -> /PCIE_DOWNSTREAM1/PCIE_TX_P
- CN1 pad B15: /PCIE_DOWNSTREAM/PCIE_TX_N -> /PCIE_DOWNSTREAM1/PCIE_TX_N
- CN1 pad B2: /PCIE_DOWNSTREAM/+12V -> /+12V_PCIE
- CN1 pad B3: /PCIE_DOWNSTREAM/+12V -> /+12V_PCIE
- CN1 pad B8: /PCIE_DOWNSTREAM/+3.3V -> /3.3V_PCIE
- CN1 pad B9: /PCIE_DOWNSTREAM/+3.3V -> /3.3V_PCIE
- J1 pad A10: /PCIE_UPSTREAM/3.3V-PCIE -> /3.3V_PCIE
- J1 pad A2: /PCIE_UPSTREAM/12V-PCIE -> /+12V_PCIE
- J1 pad A3: /PCIE_UPSTREAM/12V-PCIE -> /+12V_PCIE
- J1 pad A9: /PCIE_UPSTREAM/3.3V-PCIE -> /3.3V_PCIE
- J1 pad B1: /PCIE_UPSTREAM/12V-PCIE -> /+12V_PCIE
- J1 pad B10: /PCIE_UPSTREAM/3.3V-PCIE -> /3.3V_PCIE
- J1 pad B2: /PCIE_UPSTREAM/12V-PCIE -> /+12V_PCIE
- J1 pad B3: /PCIE_UPSTREAM/12V-PCIE -> /+12V_PCIE
- J1 pad B8: /PCIE_UPSTREAM/3.3V-PCIE -> /3.3V_PCIE
Other:
- outline, holes or cut-outs redrawn
- copper layers 2 -> 6

Commit message: Layout is finished.
Parts:
- moved LDO2 129.5 mm to (53.3, 112.7), turned to 180 degrees
- moved C39 126.7 mm to (201.2, 124.8), turned to 180 degrees
- moved C55 124.8 mm to (51.5, 110.2)
- moved LDO1 124.5 mm to (60.8, 112.7), turned to 180 degrees
- moved C47 123.7 mm to (201.2, 123.8), turned to 180 degrees
- moved U3 122.3 mm to (67.9, 112.7), turned to 180 degrees
- moved C56 121.2 mm to (54.6, 110.2), turned to 180 degrees
- moved C53 119.1 mm to (59.0, 110.2)
- moved C50 115.0 mm to (66.1, 110.2), turned to 180 degrees
- moved C54 115.0 mm to (62.6, 110.2), turned to 180 degrees
- moved U4 113.9 mm to (75.0, 112.7), turned to 180 degrees
- moved C40 113.4 mm to (187.8, 125.7)
- moved C43 113.0 mm to (187.8, 124.6)
- moved C49 112.7 mm to (69.7, 110.2)
- moved R23 109.1 mm to (187.8, 129.4), turned to 180 degrees
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Other:
- board size 8.4 x 20.3 mm -> 165.7 x 47.5 mm

Commit message: Finished with routing.
Parts:
- added R25: 0, Resistor_SMD:R_0402_1005Metric, F.Cu at (58.7, 130.8)
- added R26: 0, Resistor_SMD:R_0402_1005Metric, F.Cu at (58.7, 129.8)
- added R27: 0, Resistor_SMD:R_0402_1005Metric, F.Cu at (58.2, 135.6)
- added R28: 0, Resistor_SMD:R_0402_1005Metric, F.Cu at (58.2, 134.6)
- added R29: 0, Resistor_SMD:R_0402_1005Metric, F.Cu at (56.3, 116.4)
- added R30: 0, Resistor_SMD:R_0402_1005Metric, F.Cu at (63.7, 116.4)
- added R31: 0, Resistor_SMD:R_0402_1005Metric, F.Cu at (71.9, 116.4)
- added R32: 0, Resistor_SMD:R_0402_1005Metric, F.Cu at (49.1, 113.5)
- added R33: 0, Resistor_SMD:R_0402_1005Metric, F.Cu at (48.7, 127.7)
- moved L5 47.9 mm to (56.4, 118.3), turned to 180 degrees
- moved C24 41.2 mm to (81.6, 107.2), turned to -90 degrees
- moved C20 39.7 mm to (83.9, 107.3), turned to -90 degrees
- moved L1 31.0 mm to (84.6, 112.9), turned to -90 degrees
- moved C25 30.1 mm to (104.2, 124.4), turned to 180 degrees
- moved C17 29.6 mm to (98.7, 137.3), turned to 90 degrees
- moved C16 20.1 mm to (77.6, 126.5), turned to 180 degrees
- moved L6 14.5 mm to (83.7, 138.9), turned to -90 degrees
- moved C55 14.4 mm to (65.9, 110.1)
- moved LDO2 14.4 mm to (67.7, 112.6)
- moved C56 14.4 mm to (69.0, 110.1)
- moved C33 13.3 mm to (81.8, 138.2), turned to 180 degrees
- moved R3 9.76 mm to (92.8, 147.7), turned to 90 degrees
- moved C31 9.39 mm to (83.3, 133.2)
- moved C50 8.11 mm to (58.0, 110.2)
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Connections:
- J1 pad A11: /PCIE_SWITCH/PERST_L -> /PCIE_SWITCH/PCIE_nRST
- J1 pad A13: /PCIE_SWITCH/REFCLK(0)_N -> /PCIE_SWITCH/PCIE_CLK_N
- J1 pad A14: /PCIE_SWITCH/REFCLK(0)_P -> /PCIE_SWITCH/PCIE_CLK_P
- J1 pad A16: /PCIE_SWITCH/PER(0)_P -> /PCIE_SWITCH/PCIE_TX_P
- J1 pad A17: /PCIE_SWITCH/PER(0)_N -> /PCIE_SWITCH/PCIE_TX_N
- LDO1 pad 3: /3.3V_PCIE -> Net-(LDO1-EN)
- LDO2 pad 3: /PCIE_SWITCH/1.0Vaux -> Net-(LDO2-EN)
- U3 pad 3: /PCIE_SWITCH/3.3Vaux -> Net-(U3-EN)
- U4 pad 3: /PCIE_SWITCH/+3.3V -> Net-(U4-EN)
Routing:
- net /+12V_PCIE: track 0.00 -> 318.8 mm, vias 0 -> 7
- net /3.3V_PCIE: track 0.00 -> 298.5 mm, vias 0 -> 7
- net GND: track 0.00 -> 162.5 mm, vias 0 -> 57
- net /PCIE_SWITCH/PET(3)_P: track 0.00 -> 159.6 mm, vias 0 -> 2
- net /PCIE_SWITCH/PET(3)_N: track 0.00 -> 158.4 mm, vias 0 -> 2
- net /PCIE_SWITCH/PER(3)_N: track 0.00 -> 153.3 mm, vias 0 -> 2
- net /PCIE_SWITCH/PER(3)_P: track 0.00 -> 152.0 mm, vias 0 -> 3
- net /PCIE_SWITCH/DWNRST_L(3): track 0.00 -> 146.7 mm, vias 0 -> 5
- net /PCIE_SWITCH/3.3V_PCIE: track 0.00 -> 138.0 mm, vias 0 -> 13
- net /PCIE_SWITCH/PET(2)_N: track 0.00 -> 134.6 mm, vias 0 -> 2
- net /PCIE_SWITCH/PET(2)_P: track 0.00 -> 134.2 mm, vias 0 -> 2
- net /PCIE_SWITCH/PER(2)_P: track 0.00 -> 120.4 mm, vias 0 -> 1
- net /PCIE_SWITCH/REFCLK(3)_P: track 0.00 -> 118.2 mm, vias 0 -> 2
- net /PCIE_SWITCH/REFCLK(3)_N: track 0.00 -> 117.7 mm, vias 0 -> 2
- net /PCIE_SWITCH/PER(2)_N: track 0.00 -> 116.9 mm, vias 0 -> 1
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- added copper zone on B.Cu, net GND
- added copper zone on F.Cu, net GND
- added copper zone on In1.Cu, net GND
- added copper zone on In2.Cu, net GND
- added copper zone on In3.Cu, net GND
- added copper zone on In4.Cu, net GND
Other:
- board text added: "1.0V"
- board text added: "1.0vAux"
- board text added: "3.3V"
- board text added: "3.3vAux"
- board text added: "PCIE SWITCH TEST"
- board text added: "RFCLK"
- board text added: "[<-RX | TX ->]"
- board text added: "[<-TX | RX->]"
