File: switch/PCIE_SWITCH.kicad_sch (KiCad schematic)
At the start: 0 parts

Commit message: WOrking.
Parts:
- added C1, C10, C11, C14, C15, C16, C17, C19, C2, C20, C21, C22, C23, C24, C25, C26, C28, C29, C3, C30, C31, C32, C33, C4, C43, C44, C45, C46, C58, C59, C6, C60, C61, C62, C64, C65, C66, C67, C68, C69, C7, C70, C71, C8, C9: 100n, Capacitor_SMD:C_0402_1005Metric, symbol Device:C
- added C27, C57, C63: 10u, Capacitor_SMD:C_0402_1005Metric, symbol Device:C
- added L10, L11, L12, L13, L8, L9: MPZ1608D101BTA00, NEW:L0603, symbol NEW:MPZ1608D101BTA00
- added R11, R12, R13, R14, R3, R4, R8, R84, R85, R86, R87: 330, Resistor_SMD:R_0402_1005Metric, symbol Device:R
- added R15, R16, R19, R20: 5.1k, Resistor_SMD:R_0402_1005Metric, symbol Device:R
- added R2: 1.42k, Resistor_SMD:R_0402_1005Metric, symbol Device:R
- added R21, R5, R6, R7: 10k, Resistor_SMD:R_0402_1005Metric, symbol Device:R
- added R22, R23, R24: 1k, Resistor_SMD:R_0402_1005Metric, symbol Device:R
- added R88: 475, Resistor_SMD:R_0402_1005Metric, symbol Device:R
- added U1: PI7C9X2G404SLBFDEX, NEW:LQFP-128_L14.0-W14.0-P0.40-LS16.0-BL-EP5.8, symbol NEW:PI7C9X2G404SLBFDEX
- added U3: M24C04-WMN6TP, NEW:SOIC-8_L4.9-W3.9-P1.27-LS6.0-BL, symbol NEW:M24C04-WMN6TP
Connections:
- new net: R7.1, U1.44 (GPIO[7])
- new net: R12.2, U1.17 (TEST3)
- new net: R24.2, U1.21 (PRSNT[3])
- new net: R4.2, U1.53 (PL_512B)
- new net: R88.1, U1.86 (IREF)
- new net: R14.2, U1.25 (TEST5)
- new net: R21.2, U3.7 (~{WC})
- new net: R22.2, U1.19 (PRSNT[1])
- new net: R2.1, U1.116 (REXT)
- new net: R2.2, U1.115 (REXT_GND)
- new net: R13.2, U1.51 (TEST6)
- new net: R23.2, U1.20 (PRSNT[2])
- new net: R15.2, U1.16 (TEST2)
- new net: R8.1, U1.94 (TRST_L)
- new net: R6.1, U1.43 (GPIO[6])
- new net: R3.2, U1.33 (SLOTCLK)
- new net: R5.1, U1.42 (GPIO[5])
- new net: R16.2, U1.9 (TEST1)
- new net: R11.1, U1.92 (TMS)
- new net +1.0V: C28.2, C29.2, C30.2, C31.2, C32.2, C33.2, C43.2, C44.2, C45.2, C46.2, C57.2, L12.2, U1.23 (VDDC), U1.29 (VDDC), U1.3 (VDDC), U1.31 (VDDC), U1.40 (VDDC), U1.55 (VDDC), U1.62 (VDDC), U1.65 (VDDC), U1.91 (VDDC)
- new net +3.3V: L13.1
- new net +AVDD: C58.1, C59.1, C60.1, C61.1, C62.1, C63.1, L12.1, U1.105 (AVDD), U1.108 (AVDD), U1.119 (AVDD), U1.125 (AVDD), U1.99 (AVDD)
- new net +AVDDH: C70.1, L10.1, U1.113 (AVDDH)
- new net +CVDDR: C64.1, C65.1, C66.1, C67.1, L8.1, U1.79 (CVDDR), U1.82 (CVDDR), U1.84 (CVDDR)
- new net +VAUX: C71.1, L11.1, U1.15 (VAUX)
- new net +VDDCAUX: C68.1, C69.1, L9.1, U1.13 (VDDCAUX), U1.14 (VDDCAUX)
- new net 1.0Vaux: L9.2
- new net 3.3V_PCIE: C21.1, C22.1, C23.1, C24.1, C25.1, C26.1, C27.1, L10.2, L13.2, L8.2, R15.1, R16.1, R19.1, R20.1, R3.1, U1.1 (VDDR), U1.49 (VDDR), U1.64 (VDDR), U1.8 (VDDR), U1.96 (VDDR), U3.8 (VCC)
- new net 3.3Vaux: L11.2
- new net EECLK: R19.2, U1.70 (EECLK), U3.6 (SCL)
- new net EEPD: R20.2, U1.71 (EEPD), U3.5 (SDA)
- new net GND: C21.2, C22.2, C23.2, C24.2, C25.2, C26.2, C27.2, C28.1, C29.1, C30.1, C31.1, C32.1, C33.1, C43.1, C44.1, C45.1, C46.1, C57.1, C58.2, C59.2, C60.2, C61.2, C62.2, C63.2, C64.2, C65.2, C66.2, C67.2, C68.2, C69.2, C70.2, C71.2, R11.2, R12.1, R13.1, R14.1, R21.1, R22.1, R23.1, R24.1, R4.1, R5.2, R6.2, R7.2, R8.2, R84.2, R85.2, R86.2, R87.2, R88.2, U1.104 (VSS), U1.109 (CGND), U1.11 (VSS), U1.112 (CGND), U1.12 (VSS), U1.120 (VSS), U1.126 (VSS), U1.129 (EP), U1.2 (VSS), U1.30 (VSS), U1.32 (VSS), U1.34 (VSS), U1.4 (VSS), U1.41 (VSS), U1.50 (VSS), U1.56 (VSS), U1.61 (VSS), U1.63 (VSS), U1.66 (VSS), U1.87 (VSS), U1.90 (VSS), U1.95 (VSS), U3.4 (VSS)
- new net IO_SCL: U1.26 (SMBCLK)
- new net IO_SDA: U1.27 (SMBDATA)
- new net PCIE_CLK_N: U1.73 (REFCLKI_N)
- new net PCIE_CLK_P: U1.74 (REFCLKI_P)
- new net PCIE_CLK_nREQ: R87.1
- new net PCIE_RX_N: C2.1
- new net PCIE_RX_P: C1.1
- new net PCIE_TX_N: U1.127 (PERN[0])
- new net PCIE_TX_P: U1.128 (PERP[0])
- new net PCIE_nRST: U1.10 (PERST_L)
- new net PCIe_CLK_REQ(1): R86.1
- new net PCIe_CLK_REQ(2): R84.1
- new net PCIe_CLK_REQ(3): R85.1
- new net PCIe_RX_N(1): U1.98 (PERN[1])
- new net PCIe_RX_N(2): U1.103 (PERN[2])
- new net PCIe_RX_N(3): U1.121 (PERN[3])
- new net PCIe_RX_P(1): U1.97 (PERP[1])
- new net PCIe_RX_P(2): U1.102 (PERP[2])
- new net PCIe_RX_P(3): U1.122 (PERP[3])
- new net PCIe_TX_N(1): C6.2
- new net PCIe_TX_N(2): C15.2
- new net PCIe_TX_N(3): C20.2
- new net PCIe_TX_P(1): C7.2
- new net PCIe_TX_P(2): C10.2
- new net PCIe_TX_P(3): C16.2
- new net PCIe_nRST(1): U1.5 (DWNRST_L[1])
- new net PCIe_nRST(2): U1.6 (DWNRST_L[2])
- new net PCIe_nRST(3): U1.7 (DWNRST_L[3])
- new net PET(0)_N: C2.2, U1.123 (PETN[0])
- new net PET(0)_P: C1.2, U1.124 (PETP[0])
- new net PET(1)_N: C6.1, U1.101 (PETN[1])
- new net PET(1)_P: C7.1, U1.100 (PETP[1])
- new net PET(2)_N: C15.1, U1.107 (PETN[2])
- new net PET(2)_P: C10.1, U1.106 (PETP[2])
- new net PET(3)_N: C20.1, U1.117 (PETN[3])
- new net PET(3)_P: C16.1, U1.118 (PETP[3])
- new net REFCLCK_N(1): C9.2
- new net REFCLCK_N(2): C11.2
- new net REFCLCK_N(3): C17.2
- new net REFCLCK_P(1): C8.2
- new net REFCLCK_P(2): C14.2
- new net REFCLCK_P(3): C19.2
- new net REFCLK(1)_N: C9.1, U1.80 (REFCLKO_N[1])
- new net REFCLK(1)_P: C8.1, U1.81 (REFCLKO_P[1])
- new net REFCLK(2)_N: C11.1, U1.77 (REFCLKO_N[2])
- new net REFCLK(2)_P: C14.1, U1.78 (REFCLKO_P[2])
- new net REFCLK(3)_N: C17.1, U1.75 (REFCLKO_N[3])
- new net REFCLK(3)_P: C19.1, U1.76 (REFCLKO_P[3])
- new net REFCLKO0_N: C3.2, U1.111 (REFCLKN)
- new net REFCLKO0_P: C4.2, U1.110 (REFCLKP)
- new net U1-REFLCOK_N: C3.1, U1.83 (REFCLKO_N[0])
- new net U1-REFLCOK_P: C4.1, U1.85 (REFCLKO_P[0])
- no-connect marks 0 -> 27
Other:
- removed sheet PCIE_SW_IC
- note added: "EEPROM"
- note added: "FROM RPI"
- note added: "PORT 1"
- note added: "PORT 2"
- note added: "PORT 3"
- note added: "Power Filtering"

Commit message: Finished with routing.
Parts:
- added R25, R26, R27, R28, R33: 0, Resistor_SMD:R_0402_1005Metric, symbol Device:R
Connections:
- net PCIE_CLK_N: now also R25.1; no longer U1.73 (REFCLKI_N)
- net PCIE_CLK_P: now also R26.1; no longer U1.74 (REFCLKI_P)
- net PCIE_TX_N: now also R28.1; no longer U1.127 (PERN[0])
- net PCIE_TX_P: now also R27.1; no longer U1.128 (PERP[0])
- net PCIE_nRST: now also R33.1; no longer U1.10 (PERST_L)
- new net PER(0)_N: R28.2, U1.127 (PERN[0])
- new net PER(0)_P: R27.2, U1.128 (PERP[0])
- new net PERST_L: R33.2, U1.10 (PERST_L)
- new net REFCLK(0)_N: R25.2, U1.73 (REFCLKI_N)
- new net REFCLK(0)_P: R26.2, U1.74 (REFCLKI_P)
Changed lines of the file:
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@@
     (stroke (width 0) (type default))
   )
+  (wire (pts (xy 151.13 71.12) (xy 163.83 71.12))
+    (stroke (width 0) (type default))
+  )
   (wire (pts (xy 173.99 344.17) (xy 180.34 344.17))
     (stroke (width 0) (type default))
@@
     (stroke (width 0) (type default))
   )
-  (wire (pts (xy 163.83 71.12) (xy 137.16 71.12))
-    (stroke (width 0) (type default))
-  )
   (wire (pts (xy 114.3 320.04) (xy 120.65 320.04))
     (stroke (width 0) (type default))
@@
     (stroke (width 0) (type default))
   )
+  (wire (pts (xy 143.51 71.12) (xy 137.16 71.12))
+    (stroke (width 0) (type default))
+  )
   (wire (pts (xy 233.68 119.38) (xy 233.68 121.92))
     (stroke (width 0) (type default))
@@
     (effects (font (size 1.27 1.27)) (justify right bottom))
   )
-  (label "REFCLK(0)_P" (at 163.83 83.82 0) (fields_autoplaced)
-    (effects (font (size 1.27 1.27)) (justify left bottom))
-  )
   (label "REFCLKO0_P" (at 321.31 119.38 0) (fields_autoplaced)
     (effects (font (size 1.27 1.27)) (justify left bottom))
@@
     (effects (font (size 1.27 1.27)) (justify left bottom))
   )
+  (label "PER(0)_P" (at 171.45 104.14 0) (fields_autoplaced)
+    (effects (font (size 1.27 1.27)) (justify left bottom))
+  )
   (label "U1-REFLCOK_P" (at 328.93 182.88 0) (fields_autoplaced)
     (effects (font (size 1.27 1.27)) (justify left bottom))
@@
     (effects (font (size 1.27 1.27)) (justify left bottom))
   )
+  (label "REFCLK(0)_P" (at 171.45 83.82 0) (fields_autoplaced)
+    (effects (font (size 1.27 1.27)) (justify left bottom))
+  )
   (label "REFCLK(1)_P" (at 321.31 193.04 0) (fields_autoplaced)
     (effects (font (size 1.27 1.27)) (justify left bottom))
@@
     (effects (font (size 1.27 1.27)) (justify left bottom))
   )
-  (label "PER(0)_P" (at 163.83 104.14 0) (fields_autoplaced)
-    (effects (font (size 1.27 1.27)) (justify left bottom))
-  )
   (label "PET(3)_N" (at 411.48 205.74 180) (fields_autoplaced)
     (effects (font (size 1.27 1.27)) (justify right bottom))
   )
-  (label "REFCLK(0)_N" (at 163.83 86.36 0) (fields_autoplaced)
-    (effects (font (size 1.27 1.27)) (justify left bottom))
-  )
   (label "CLOCKREQ_(0)" (at 195.58 77.47 0) (fields_autoplaced)
     (effects (font (size 1.27 1.27)) (justify left bottom))
@@
     (effects (font (size 1.27 1.27)) (justify left bottom))
   )
-  (label "PER(0)_N" (at 163.83 106.68 0) (fields_autoplaced)
-    (effects (font (size 1.27 1.27)) (justify left bottom))
-  )
   (label "IO_SCL" (at 163.83 113.03 0) (fields_autoplaced)
     (effects (font (size 1.27 1.27)) (justify left bottom))
@@
     (effects (font (size 1.27 1.27)) (justify right bottom))
   )
+  (label "PER(0)_N" (at 171.45 106.68 0) (fields_autoplaced)
+    (effects (font (size 1.27 1.27)) (justify left bottom))
+  )
   (label "PER(1)_P" (at 321.31 152.4 0) (fields_autoplaced)
     (effects (font (size 1.27 1.27)) (justify left bottom))
@@
     (effects (font (size 1.27 1.27)) (justify left bottom))
   )
+  (label "REFCLK(0)_N" (at 171.45 86.36 0) (fields_autoplaced)
+    (effects (font (size 1.27 1.27)) (justify left bottom))
+  )
   (label "PER(2)_N" (at 397.51 151.13 180) (fields_autoplaced)
     (effects (font (size 1.27 1.27)) (justify right bottom))
@@
     )
   )
+  (symbol (lib_id "Device:R") (at 167.64 104.14 90) (unit 1)
+    (in_bom yes) (on_board yes) (dnp no)
+    (property "Reference" "R27" (at 167.64 104.14 90)
+      (effects (font (size 1.27 1.27)))
+    )
+    (property "Value" "0" (at 162.56 104.14 90)
+      (effects (font (size 1.27 1.27)))
+    )
+    (property "Footprint" "Resistor_SMD:R_0402_1005Metric" (at 167.64 105.918 90)
+      (effects (font (size 1.27 1.27)) hide)
+    )
+    (property "Datasheet" "~" (at 167.64 104.14 0)
+      (effects (font (size 1.27 1.27)) hide)
+    )
+    (pin "1")
+    (pin "2")
+    (instances
+      (project "switch"
+        (path "/bb24befe-87e3-4bdd-b50d-d3887bf8bcae/786f20ee-ac35-4533-ab85-c31995b4cba5"
+          (reference "R27") (unit 1)
+        )
+      )
+    )
+  )
+  (symbol (lib_id "Device:R") (at 147.32 71.12 90) (unit 1)
+    (in_bom yes) (on_board yes) (dnp no)
+    (property "Reference" "R33" (at 147.32 71.12 90)
+      (effects (font (size 1.27 1.27)))
+    )
+    (property "Value" "0" (at 142.24 71.12 90)
+      (effects (font (size 1.27 1.27)))
+    )
+    (property "Footprint" "Resistor_SMD:R_0402_1005Metric" (at 147.32 72.898 90)
+      (effects (font (size 1.27 1.27)) hide)
+    )
+    (property "Datasheet" "~" (at 147.32 71.12 0)
+      (effects (font (size 1.27 1.27)) hide)
+    )
+    (pin "1")
+    (pin "2")
+    (instances
+      (project "switch"
+        (path "/bb24befe-87e3-4bdd-b50d-d3887bf8bcae/786f20ee-ac35-4533-ab85-c31995b4cba5"
+          (reference "R33") (unit 1)
+        )
+      )
+    )
+  )
   (symbol (lib_id "NEW:MPZ1608D101BTA00") (at 143.51 314.96 90) (unit 1)
     (in_bom yes) (on_board yes) (dnp no) (fields_autoplaced)
@@
     )
   )
+  (symbol (lib_id "Device:R") (at 167.64 106.68 90) (unit 1)
+    (in_bom yes) (on_board yes) (dnp no)
+    (property "Reference" "R28" (at 167.64 106.68 90)
+      (effects (font (size 1.27 1.27)))
+    )
+    (property "Value" "0" (at 162.56 106.68 90)
+      (effects (font (size 1.27 1.27)))
+    )
+    (property "Footprint" "Resistor_SMD:R_0402_1005Metric" (at 167.64 108.458 90)
+      (effects (font (size 1.27 1.27)) hide)
+    )
+    (property "Datasheet" "~" (at 167.64 106.68 0)
+      (effects (font (size 1.27 1.27)) hide)
+    )
+    (pin "1")
+    (pin "2")
+    (instances
+      (project "switch"
+        (path "/bb24befe-87e3-4bdd-b50d-d3887bf8bcae/786f20ee-ac35-4533-ab85-c31995b4cba5"
+          (reference "R28") (unit 1)
+        )
+      )
+    )
+  )
   (symbol (lib_id "Device:R") (at 213.36 134.62 90) (unit 1)
     (in_bom yes) (on_board yes) (dnp no)
@@
     )
   )
+  (symbol (lib_id "Device:R") (at 167.64 86.36 90) (unit 1)
+    (in_bom yes) (on_board yes) (dnp no)
+    (property "Reference" "R25" (at 167.64 86.36 90)
+      (effects (font (size 1.27 1.27)))
+    )
+    (property "Value" "0" (at 162.56 86.36 90)
+      (effects (font (size 1.27 1.27)))
+    )
+    (property "Footprint" "Resistor_SMD:R_0402_1005Metric" (at 167.64 88.138 90)
+      (effects (font (size 1.27 1.27)) hide)
+    )
+    (property "Datasheet" "~" (at 167.64 86.36 0)
+      (effects (font (size 1.27 1.27)) hide)
+    )
+    (pin "1")
+    (pin "2")
+    (instances
+      (project "switch"
+        (path "/bb24befe-87e3-4bdd-b50d-d3887bf8bcae/786f20ee-ac35-4533-ab85-c31995b4cba5"
+          (reference "R25") (unit 1)
+        )
+      )
+    )
+  )
   (symbol (lib_id "Device:R") (at 190.5 73.66 180) (unit 1)
     (in_bom yes) (on_board yes) (dnp no) (fields_autoplaced)
@@
         )
       )
+    )
+  )
+  (symbol (lib_id "Device:R") (at 167.64 83.82 90) (unit 1)
+    (in_bom yes) (on_board yes) (dnp no)
+    (property "Reference" "R26" (at 167.64 83.82 90)
+      (effects (font (size 1.27 1.27)))
+    )
+    (property "Value" "0" (at 162.56 83.82 90)
+      (effects (font (size 1.27 1.27)))
+    )
+    (property "Footprint" "Resistor_SMD:R_0402_1005Metric" (at 167.64 85.598 90)
+      (effects (font (size 1.27 1.27)) hide)
+    )
+    (property "Datasheet" "~" (at 167.64 83.82 0)
+      (effects (font (size 1.27 1.27)) hide)
+    )
+    (pin "1")
+    (pin "2")
+    (instances
+      (project "switch"
+        (path "/bb24befe-87e3-4bdd-b50d-d3887bf8bcae/786f20ee-ac35-4533-ab85-c31995b4cba5"
+          (reference "R26") (unit 1)
+        )
+      )

Commit message: Added Production files.
Parts:
- R25, R26, R27, R28, R33: LCSC Part (none) -> C4044221
- R84, R85, R86, R87, R88: LCSC Part (none) -> C25104
Changed lines of the file:
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@@
       (effects (font (size 1.27 1.27)) hide)
     )
+    (property "LCSC Part" "C4044221" (at 167.64 104.14 0)
+      (effects (font (size 1.27 1.27)) hide)
+    )
     (pin "1")
     (pin "2")
@@
       (effects (font (size 1.27 1.27)) hide)
     )
+    (property "LCSC Part" "C4044221" (at 147.32 71.12 0)
+      (effects (font (size 1.27 1.27)) hide)
+    )
     (pin "1")
     (pin "2")
@@
       (effects (font (size 1.27 1.27)) hide)
     )
+    (property "LCSC Part" "C25104" (at 426.72 114.3 0)
+      (effects (font (size 1.27 1.27)) hide)
+    )
     (pin "1")
     (pin "2")
@@
       (effects (font (size 1.27 1.27)) hide)
     )
+    (property "LCSC Part" "C25104" (at 322.58 180.34 0)
+      (effects (font (size 1.27 1.27)) hide)
+    )
     (pin "1")
     (pin "2")
@@
       (effects (font (size 1.27 1.27)) hide)
     )
+    (property "LCSC Part" "C25104" (at 429.26 238.76 0)
+      (effects (font (size 1.27 1.27)) hide)
+    )
     (pin "1")
     (pin "2")
@@
       (effects (font (size 1.27 1.27)) hide)
     )
+    (property "LCSC Part" "C25104" (at 427.99 176.53 0)
+      (effects (font (size 1.27 1.27)) hide)
+    )
     (pin "1")
     (pin "2")
@@
       (effects (font (size 1.27 1.27)) hide)
     )
+    (property "LCSC Part" "C4044221" (at 167.64 106.68 0)
+      (effects (font (size 1.27 1.27)) hide)
+    )
     (pin "1")
     (pin "2")
@@
       (effects (font (size 1.27 1.27)) hide)
     )
+    (property "LCSC Part" "C4044221" (at 167.64 86.36 0)
+      (effects (font (size 1.27 1.27)) hide)
+    )
     (pin "1")
     (pin "2")
@@
       (effects (font (size 1.27 1.27)) hide)
     )
+    (property "LCSC Part" "C25104" (at 190.5 73.66 0)
+      (effects (font (size 1.27 1.27)) hide)
+    )
     (pin "1")
     (pin "2")
@@
       (effects (font (size 1.27 1.27)) hide)
     )
+    (property "LCSC Part" "C4044221" (at 167.64 83.82 0)
+      (effects (font (size 1.27 1.27)) hide)
+    )
