File: switch/SW_PSU.kicad_sch (KiCad schematic)
At the start: 12 parts, among them U3 TLV73310PDBVR, U4 TLV73310PDBVR

Commit message: Finished with routing.
Parts:
- added R28 (x4): 0, Resistor_SMD:R_0402_1005Metric, symbol Device:R
Connections:
- net 1.0VAux: now also R28.2; no longer LDO2.3 (EN)
- net 3.3V: now also R28.2; no longer U4.3 (EN)
- net 3.3VAux: now also R28.2; no longer U3.3 (EN)
- net 3.3VPcie: now also R28.1; no longer LDO1.3 (EN)
- new net: R28.1, U4.3 (EN)
- new net: LDO1.3 (EN), R28.2
- new net: R28.1, U3.3 (EN)
- new net: LDO2.3 (EN), R28.1
Changed lines of the file:
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@@
 (kicad_sch (version 20230121) (generator eeschema)
   (paper "A4")
+  (junction (at 132.08 74.93) (diameter 0) (color 0 0 0 0)
+  )
+  (junction (at 36.83 52.07) (diameter 0) (color 0 0 0 0)
+  )
+  (junction (at 181.61 100.33) (diameter 0) (color 0 0 0 0)
+  )
+  (junction (at 214.63 125.73) (diameter 0) (color 0 0 0 0)
+  )
+  (junction (at 149.86 100.33) (diameter 0) (color 0 0 0 0)
+  )
   (junction (at 182.88 100.33) (diameter 0) (color 0 0 0 0)
-  )
-  (junction (at 130.81 74.93) (diameter 0) (color 0 0 0 0)
-  )
-  (junction (at 73.66 52.07) (diameter 0) (color 0 0 0 0)
-  )
-  (junction (at 36.83 52.07) (diameter 0) (color 0 0 0 0)
-  )
-  (junction (at 181.61 100.33) (diameter 0) (color 0 0 0 0)
-  )
-  (junction (at 214.63 125.73) (diameter 0) (color 0 0 0 0)
-  )
-  (junction (at 149.86 100.33) (diameter 0) (color 0 0 0 0)
   )
   (junction (at 93.98 73.66) (diameter 0) (color 0 0 0 0)
@@
   (no_connect (at 237.49 129.54))
   (no_connect (at 176.53 105.41))
+  (wire (pts (xy 252.73 127) (xy 248.92 127))
+    (stroke (width 0) (type default))
+  )
+  (wire (pts (xy 182.88 123.19) (xy 182.88 100.33))
+    (stroke (width 0) (type default))
+  )
+  (wire (pts (xy 121.92 74.93) (xy 132.08 74.93))
+    (stroke (width 0) (type default))
+  )
+  (wire (pts (xy 36.83 57.15) (xy 38.1 57.15))
+    (stroke (width 0) (type default))
+  )
+  (wire (pts (xy 36.83 52.07) (xy 39.37 52.07))
+    (stroke (width 0) (type default))
+  )
+  (wire (pts (xy 248.92 127) (xy 237.49 127))
+    (stroke (width 0) (type default))
+  )
+  (wire (pts (xy 71.12 52.07) (xy 66.04 52.07))
+    (stroke (width 0) (type default))
+  )
+  (wire (pts (xy 149.86 100.33) (xy 156.21 100.33))
+    (stroke (width 0) (type default))
+  )
   (wire (pts (xy 182.88 130.81) (xy 217.17 130.81))
     (stroke (width 0) (type default))
   )
-  (wire (pts (xy 130.81 105.41) (xy 156.21 105.41))
-    (stroke (width 0) (type default))
-  )
-  (wire (pts (xy 252.73 127) (xy 248.92 127))
-    (stroke (width 0) (type default))
-  )
-  (wire (pts (xy 130.81 74.93) (xy 130.81 105.41))
-    (stroke (width 0) (type default))
-  )
-  (wire (pts (xy 73.66 78.74) (xy 73.66 52.07))
-    (stroke (width 0) (type default))
-  )
-  (wire (pts (xy 130.81 74.93) (xy 121.92 74.93))
-    (stroke (width 0) (type default))
-  )
-  (wire (pts (xy 36.83 52.07) (xy 39.37 52.07))
+  (wire (pts (xy 116.84 74.93) (xy 121.92 74.93))
+    (stroke (width 0) (type default))
+  )
+  (wire (pts (xy 132.08 74.93) (xy 134.62 74.93))
     (stroke (width 0) (type default))
   )
@@
     (stroke (width 0) (type default))
   )
-  (wire (pts (xy 248.92 127) (xy 237.49 127))
-    (stroke (width 0) (type default))
-  )
-  (wire (pts (xy 71.12 52.07) (xy 66.04 52.07))
-    (stroke (width 0) (type default))
-  )
-  (wire (pts (xy 36.83 57.15) (xy 45.72 57.15))
-    (stroke (width 0) (type default))
-  )
-  (wire (pts (xy 149.86 100.33) (xy 156.21 100.33))
-    (stroke (width 0) (type default))
-  )
-  (wire (pts (xy 116.84 74.93) (xy 121.92 74.93))
+  (wire (pts (xy 132.08 87.63) (xy 132.08 74.93))
+    (stroke (width 0) (type default))
+  )
+  (wire (pts (xy 147.32 100.33) (xy 149.86 100.33))
+    (stroke (width 0) (type default))
+  )
+  (wire (pts (xy 210.82 125.73) (xy 214.63 125.73))
+    (stroke (width 0) (type default))
+  )
+  (wire (pts (xy 71.12 52.07) (xy 74.93 52.07))
+    (stroke (width 0) (type default))
+  )
+  (wire (pts (xy 214.63 125.73) (xy 217.17 125.73))
+    (stroke (width 0) (type default))
+  )
+  (wire (pts (xy 181.61 100.33) (xy 176.53 100.33))
+    (stroke (width 0) (type default))
+  )
+  (wire (pts (xy 91.44 73.66) (xy 93.98 73.66))
     (stroke (width 0) (type default))
   )
@@
     (stroke (width 0) (type default))
   )
-  (wire (pts (xy 147.32 100.33) (xy 149.86 100.33))
-    (stroke (width 0) (type default))
-  )
-  (wire (pts (xy 210.82 125.73) (xy 214.63 125.73))
-    (stroke (width 0) (type default))
-  )
-  (wire (pts (xy 71.12 52.07) (xy 73.66 52.07))
-    (stroke (width 0) (type default))
-  )
-  (wire (pts (xy 214.63 125.73) (xy 217.17 125.73))
-    (stroke (width 0) (type default))
-  )
-  (wire (pts (xy 181.61 100.33) (xy 176.53 100.33))
-    (stroke (width 0) (type default))
-  )
-  (wire (pts (xy 182.88 100.33) (xy 182.88 130.81))
-    (stroke (width 0) (type default))
-  )
-  (wire (pts (xy 91.44 73.66) (xy 93.98 73.66))
-    (stroke (width 0) (type default))
-  )
-  (wire (pts (xy 134.62 74.93) (xy 130.81 74.93))
+  (wire (pts (xy 132.08 95.25) (xy 132.08 105.41))
+    (stroke (width 0) (type default))
+  )
+  (wire (pts (xy 71.12 52.07) (xy 71.12 71.12))
     (stroke (width 0) (type default))
   )
@@
     (stroke (width 0) (type default))
   )
-  (wire (pts (xy 73.66 52.07) (xy 74.93 52.07))
-    (stroke (width 0) (type default))
-  )
   (wire (pts (xy 39.37 52.07) (xy 45.72 52.07))
     (stroke (width 0) (type default))
   )
-  (wire (pts (xy 96.52 78.74) (xy 73.66 78.74))
+  (wire (pts (xy 132.08 105.41) (xy 156.21 105.41))
+    (stroke (width 0) (type default))
+  )
+  (wire (pts (xy 96.52 78.74) (xy 71.12 78.74))
     (stroke (width 0) (type default))
   )
@@
   (hierarchical_label "3.3V" (shape output) (at 185.42 100.33 0) (fields_autoplaced)
     (effects (font (size 1.27 1.27)) (justify left))
+  )
+  (symbol (lib_id "Device:R") (at 182.88 127 180) (unit 1)
+    (in_bom yes) (on_board yes) (dnp no)
+    (property "Reference" "R28" (at 182.88 127 90)
+      (effects (font (size 1.27 1.27)))
+    )
+    (property "Value" "0" (at 182.88 132.08 90)
+      (effects (font (size 1.27 1.27)))
+    )
+    (property "Footprint" "Resistor_SMD:R_0402_1005Metric" (at 184.658 127 90)
+      (effects (font (size 1.27 1.27)) hide)
+    )
+    (property "Datasheet" "~" (at 182.88 127 0)
+      (effects (font (size 1.27 1.27)) hide)
+    )
+    (pin "1")
+    (pin "2")
+    (instances
+      (project "switch"
+        (path "/bb24befe-87e3-4bdd-b50d-d3887bf8bcae/786f20ee-ac35-4533-ab85-c31995b4cba5"
+          (reference "R28") (unit 1)
+        )
+        (path "/bb24befe-87e3-4bdd-b50d-d3887bf8bcae/b792fb4a-116f-4d37-b812-23a041b1618b"
+          (reference "R31") (unit 1)
+        )
+      )
+    )
   )
   (symbol (lib_id "NEW:TPS70933DBVR") (at 55.88 54.61 0) (unit 1)
@@
     )
   )
+  (symbol (lib_id "Device:R") (at 41.91 57.15 90) (unit 1)
+    (in_bom yes) (on_board yes) (dnp no)
+    (property "Reference" "R28" (at 41.91 57.15 90)
+      (effects (font (size 1.27 1.27)))
+    )
+    (property "Value" "0" (at 36.83 57.15 90)
+      (effects (font (size 1.27 1.27)))
+    )
+    (property "Footprint" "Resistor_SMD:R_0402_1005Metric" (at 41.91 58.928 90)
+      (effects (font (size 1.27 1.27)) hide)
+    )
+    (property "Datasheet" "~" (at 41.91 57.15 0)
+      (effects (font (size 1.27 1.27)) hide)
+    )
+    (pin "1")
+    (pin "2")
+    (instances
+      (project "switch"
+        (path "/bb24befe-87e3-4bdd-b50d-d3887bf8bcae/786f20ee-ac35-4533-ab85-c31995b4cba5"
+          (reference "R28") (unit 1)
+        )
+        (path "/bb24befe-87e3-4bdd-b50d-d3887bf8bcae/b792fb4a-116f-4d37-b812-23a041b1618b"
+          (reference "R32") (unit 1)
+        )
+      )
+    )
+  )
   (symbol (lib_id "Device:C") (at 248.92 130.81 0) (unit 1)
     (in_bom yes) (on_board yes) (dnp no) (fields_autoplaced)
@@
     )
   )
+  (symbol (lib_id "Device:R") (at 132.08 91.44 180) (unit 1)
+    (in_bom yes) (on_board yes) (dnp no)
+    (property "Reference" "R28" (at 132.08 91.44 90)
+      (effects (font (size 1.27 1.27)))
+    )
+    (property "Value" "0" (at 132.08 96.52 90)
+      (effects (font (size 1.27 1.27)))
+    )
+    (property "Footprint" "Resistor_SMD:R_0402_1005Metric" (at 133.858 91.44 90)
+      (effects (font (size 1.27 1.27)) hide)
+    )
+    (property "Datasheet" "~" (at 132.08 91.44 0)
+      (effects (font (size 1.27 1.27)) hide)
+    )
+    (pin "1")
+    (pin "2")
+    (instances
+      (project "switch"
+        (path "/bb24befe-87e3-4bdd-b50d-d3887bf8bcae/786f20ee-ac35-4533-ab85-c31995b4cba5"
+          (reference "R28") (unit 1)
+        )
+        (path "/bb24befe-87e3-4bdd-b50d-d3887bf8bcae/b792fb4a-116f-4d37-b812-23a041b1618b"
+          (reference "R30") (unit 1)
+        )
+      )
+    )
+  )
   (symbol (lib_id "power:GND") (at 181.61 92.71 180) (unit 1)
     (in_bom yes) (on_board yes) (dnp no) (fields_autoplaced)
@@
         )
       )
+    )
+  )
+  (symbol (lib_id "Device:R") (at 71.12 74.93 0) (mirror x) (unit 1)
+    (in_bom yes) (on_board yes) (dnp no)
+    (property "Reference" "R28" (at 71.12 74.93 90)
+      (effects (font (size 1.27 1.27)))
+    )
+    (property "Value" "0" (at 71.12 80.01 90)
+      (effects (font (size 1.27 1.27)))
+    )
+    (property "Footprint" "Resistor_SMD:R_0402_1005Metric" (at 69.342 74.93 90)
+      (effects (font (size 1.27 1.27)) hide)
+    )
+    (property "Datasheet" "~" (at 71.12 74.93 0)
+      (effects (font (size 1.27 1.27)) hide)
+    )
+    (pin "1")
+    (pin "2")
+    (instances
+      (project "switch"
+        (path "/bb24befe-87e3-4bdd-b50d-d3887bf8bcae/786f20ee-ac35-4533-ab85-c31995b4cba5"
+          (reference "R28") (unit 1)
+        )
+        (path "/bb24befe-87e3-4bdd-b50d-d3887bf8bcae/b792fb4a-116f-4d37-b812-23a041b1618b"
+          (reference "R29") (unit 1)
+        )
+      )

Commit message: Added Production files.
Parts:
- C49, C50, C51, C52, C53, C55: LCSC Part (none) -> C77006
- C54, C56: LCSC Part (none) -> C694168
- R28: LCSC Part (none) -> C4044221
Changed lines of the file:
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@@
+      (effects (font (size 1.27 1.27)) hide)
+    )
+    (property "LCSC Part" "C4044221" (at 182.88 127 0)
       (effects (font (size 1.27 1.27)) hide)
     )
@@
       (effects (font (size 1.27 1.27)) hide)
     )
+    (property "LCSC Part" "C4044221" (at 41.91 57.15 0)
+      (effects (font (size 1.27 1.27)) hide)
+    )
     (pin "1")
     (pin "2")
@@
       (effects (font (size 1.27 1.27)) hide)
     )
+    (property "LCSC Part" "C77006" (at 248.92 130.81 0)
+      (effects (font (size 1.27 1.27)) hide)
+    )
     (pin "1")
     (pin "2")
@@
     )
     (property "Datasheet" "~" (at 181.61 96.52 0)
+      (effects (font (size 1.27 1.27)) hide)
+    )
+    (property "LCSC Part" "C694168" (at 181.61 96.52 0)
       (effects (font (size 1.27 1.27)) hide)
     )
@@
       (effects (font (size 1.27 1.27)) hide)
     )
+    (property "LCSC Part" "C77006" (at 93.98 69.85 0)
+      (effects (font (size 1.27 1.27)) hide)
+    )
     (pin "1")
     (pin "2")
@@
       (effects (font (size 1.27 1.27)) hide)
     )
+    (property "LCSC Part" "C77006" (at 149.86 96.52 0)
+      (effects (font (size 1.27 1.27)) hide)
+    )
     (pin "1")
     (pin "2")
@@
     )
     (property "Datasheet" "~" (at 214.63 121.92 0)
+      (effects (font (size 1.27 1.27)) hide)
+    )
+    (property "LCSC Part" "C77006" (at 214.63 121.92 0)
       (effects (font (size 1.27 1.27)) hide)
     )
@@
       (effects (font (size 1.27 1.27)) hide)
     )
+    (property "LCSC Part" "C4044221" (at 132.08 91.44 0)
+      (effects (font (size 1.27 1.27)) hide)
+    )
     (pin "1")
     (pin "2")
@@
       (effects (font (size 1.27 1.27)) hide)
     )
+    (property "LCSC Part" "C77006" (at 39.37 48.26 0)
+      (effects (font (size 1.27 1.27)) hide)
+    )
     (pin "1")
     (pin "2")
@@
       (effects (font (size 1.27 1.27)) hide)
     )
+    (property "LCSC Part" "C77006" (at 121.92 78.74 0)
+      (effects (font (size 1.27 1.27)) hide)
+    )
     (pin "1")
     (pin "2")
@@
     )
     (property "Datasheet" "~" (at 71.12 48.26 0)
+      (effects (font (size 1.27 1.27)) hide)
+    )
+    (property "LCSC Part" "C694168" (at 71.12 48.26 0)
       (effects (font (size 1.27 1.27)) hide)
     )
@@
       (effects (font (size 1.27 1.27)) hide)
     )
+    (property "LCSC Part" "C4044221" (at 71.12 74.93 0)
+      (effects (font (size 1.27 1.27)) hide)
+    )
